File: Arcjet-PPU.kicad_sch (KiCad schematic)
At the start: 32 parts, among them J1 Conn_01x02, Q5 C3M0900170D, U2 UCC27511ADBV, U3 INA180A2

Commit message: formatting
Parts:
- removed C1, C2, C3, C4, C5, C6: 100u, symbol Device:C_Polarized
- removed C11: 100n, Capacitor_SMD:C_0603_1608Metric_Pad1.08x0.95mm_HandSolder, symbol Device:C
- removed C12: 2.2u, Capacitor_SMD:C_0603_1608Metric_Pad1.08x0.95mm_HandSolder, symbol Device:C
- removed C13: 10n, Capacitor_SMD:C_0603_1608Metric_Pad1.08x0.95mm_HandSolder, symbol Device:C
- removed D10, D2, D7, D8, D9: 1.5KExxA, Diode_THT:D_DO-201AE_P15.24mm_Horizontal, symbol Diode:1.5KExxA
- removed D11: BAV199, Package_TO_SOT_SMD:SOT-23, symbol Device:D_Dual_Series_AKC
- removed J1: Conn_01x02, symbol Connector_Generic:Conn_01x02
- removed L1: 470u, symbol Device:L
- removed Q5: C3M0900170D, Package_TO_SOT_THT:TO-247-3_Vertical, symbol Device:Q_NMOS
- removed R12: 3.3, symbol Device:R
- removed R13: 0, symbol Device:R
- removed R14, R18, R19, R20: 51k, symbol Device:R
- removed R15, R17, R21: 2.2k, symbol Device:R
- removed R16: 100k, symbol Device:R
- removed R2, R3: 2m, symbol Device:R
- removed U2: UCC27511ADBV, Package_TO_SOT_SMD:SOT-23-6, symbol Driver_FET:UCC27511ADBV
- removed U3: INA180A2, Package_TO_SOT_SMD:SOT-23-5, symbol Amplifier_Current:INA180A2
Other:
- removed sheet Half Bridge
- added sheet Constant Current Supply (CCS.kicad_sch)
- added sheet IO (IO.kicad_sch)
- added sheet Micro (Micro.kicad_sch)
- note removed: "2m shunt & INA180 A2 variant saturates at 33A with 3.3v supply"
- note removed: "Capacitance?"
- note removed: "Need INA? Need protection?"
- note removed: "Need more protection?"
- note removed: "OUTPUT"
- note removed: "Resistor values?"
- note removed: "Should not be connected to an STM32 FT pin since those don't have clamping diodes"
- note removed: "TVS diodes and shunt FET picked by Claude, check"
- note removed: "These need to handle ~1.3 kV total so probably 1206 or TH"
- company: (none) -> Rutgers Capstone ECE 2026-2027
- title: (none) -> Arc Jet PU (Power Unit)
