File: Gate_Resistors.kicad_sch (KiCad schematic)
At the start: 3 parts

Commit message: formatting
Parts:
- renumbered D3 to D6, R4 to R10, R5 to R11
Other:
- company: (none) -> Rutgers Capstone ECE 2026-2027
- title: (none) -> Arc Jet PU (Power Unit)
Changed lines of the file:
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@@
 	(generator_version "10.0")
 	(paper "A4")
+	(title_block
+		(title "Arc Jet PU (Power Unit)")
+		(date "2026-10-29")
+		(rev "1.0")
+		(company "Rutgers Capstone ECE 2026-2027")
+		(comment 1 "Mark Tymoshenko mat399@scarletmail.rutgers.edu")
+		(comment 2 "Cy Westbrook")
+	)
 	(wire
 		(pts
@@
 		(in_pos_files yes)
 		(dnp no)
-		(property "Reference" "R5"
+		(property "Reference" "R11"
 			(at 151.13 87.884 90)
 			(show_name no)
@@
 		(instances
 			(project "Arcjet-PPU"
-				(path "/a26094a8-870e-4d79-a298-19a2c7b26655/1ff5d421-dfac-490f-b230-bb532702cb90/1462f3fc-c77a-4020-babf-9c1e874adae4"
+				(path "/a26094a8-870e-4d79-a298-19a2c7b26655/3b902dd1-f160-4711-ad5c-803c38714d8b/8b541bd0-7703-41c7-b1bc-19a6eec4959f/1462f3fc-c77a-4020-babf-9c1e874adae4"
 					(reference "R11")
 					(unit 1)
 				)
-				(path "/a26094a8-870e-4d79-a298-19a2c7b26655/1ff5d421-dfac-490f-b230-bb532702cb90/6ed8d3e8-172a-454e-91a1-212a5b405cd8"
+				(path "/a26094a8-870e-4d79-a298-19a2c7b26655/3b902dd1-f160-4711-ad5c-803c38714d8b/8b541bd0-7703-41c7-b1bc-19a6eec4959f/6ed8d3e8-172a-454e-91a1-212a5b405cd8"
 					(reference "R7")
 					(unit 1)
 				)
-				(path "/a26094a8-870e-4d79-a298-19a2c7b26655/1ff5d421-dfac-490f-b230-bb532702cb90/95a68da6-4437-469b-a050-26966337937e"
+				(path "/a26094a8-870e-4d79-a298-19a2c7b26655/3b902dd1-f160-4711-ad5c-803c38714d8b/8b541bd0-7703-41c7-b1bc-19a6eec4959f/95a68da6-4437-469b-a050-26966337937e"
 					(reference "R9")
 					(unit 1)
 				)
-				(path "/a26094a8-870e-4d79-a298-19a2c7b26655/1ff5d421-dfac-490f-b230-bb532702cb90/cf5b497f-d460-45bc-b512-00017b3e4ab3"
+				(path "/a26094a8-870e-4d79-a298-19a2c7b26655/3b902dd1-f160-4711-ad5c-803c38714d8b/8b541bd0-7703-41c7-b1bc-19a6eec4959f/cf5b497f-d460-45bc-b512-00017b3e4ab3"
 					(reference "R5")
 					(unit 1)
@@
 		(in_pos_files yes)
 		(dnp no)
-		(property "Reference" "D3"
+		(property "Reference" "D6"
 			(at 156.21 78.486 0)
 			(show_name no)
@@
 		(instances
 			(project "Arcjet-PPU"
-				(path "/a26094a8-870e-4d79-a298-19a2c7b26655/1ff5d421-dfac-490f-b230-bb532702cb90/1462f3fc-c77a-4020-babf-9c1e874adae4"
+				(path "/a26094a8-870e-4d79-a298-19a2c7b26655/3b902dd1-f160-4711-ad5c-803c38714d8b/8b541bd0-7703-41c7-b1bc-19a6eec4959f/1462f3fc-c77a-4020-babf-9c1e874adae4"
 					(reference "D6")
 					(unit 1)
 				)
-				(path "/a26094a8-870e-4d79-a298-19a2c7b26655/1ff5d421-dfac-490f-b230-bb532702cb90/6ed8d3e8-172a-454e-91a1-212a5b405cd8"
+				(path "/a26094a8-870e-4d79-a298-19a2c7b26655/3b902dd1-f160-4711-ad5c-803c38714d8b/8b541bd0-7703-41c7-b1bc-19a6eec4959f/6ed8d3e8-172a-454e-91a1-212a5b405cd8"
 					(reference "D4")
 					(unit 1)
 				)
-				(path "/a26094a8-870e-4d79-a298-19a2c7b26655/1ff5d421-dfac-490f-b230-bb532702cb90/95a68da6-4437-469b-a050-26966337937e"
+				(path "/a26094a8-870e-4d79-a298-19a2c7b26655/3b902dd1-f160-4711-ad5c-803c38714d8b/8b541bd0-7703-41c7-b1bc-19a6eec4959f/95a68da6-4437-469b-a050-26966337937e"
 					(reference "D5")
 					(unit 1)
 				)
-				(path "/a26094a8-870e-4d79-a298-19a2c7b26655/1ff5d421-dfac-490f-b230-bb532702cb90/cf5b497f-d460-45bc-b512-00017b3e4ab3"
+				(path "/a26094a8-870e-4d79-a298-19a2c7b26655/3b902dd1-f160-4711-ad5c-803c38714d8b/8b541bd0-7703-41c7-b1bc-19a6eec4959f/cf5b497f-d460-45bc-b512-00017b3e4ab3"
 					(reference "D3")
 					(unit 1)
@@
 		(in_pos_files yes)
 		(dnp no)
-		(property "Reference" "R4"
+		(property "Reference" "R10"
 			(at 143.51 78.994 90)
 			(show_name no)
@@
 		(instances
 			(project "Arcjet-PPU"
-				(path "/a26094a8-870e-4d79-a298-19a2c7b26655/1ff5d421-dfac-490f-b230-bb532702cb90/1462f3fc-c77a-4020-babf-9c1e874adae4"
+				(path "/a26094a8-870e-4d79-a298-19a2c7b26655/3b902dd1-f160-4711-ad5c-803c38714d8b/8b541bd0-7703-41c7-b1bc-19a6eec4959f/1462f3fc-c77a-4020-babf-9c1e874adae4"
 					(reference "R10")
 					(unit 1)
 				)
-				(path "/a26094a8-870e-4d79-a298-19a2c7b26655/1ff5d421-dfac-490f-b230-bb532702cb90/6ed8d3e8-172a-454e-91a1-212a5b405cd8"
+				(path "/a26094a8-870e-4d79-a298-19a2c7b26655/3b902dd1-f160-4711-ad5c-803c38714d8b/8b541bd0-7703-41c7-b1bc-19a6eec4959f/6ed8d3e8-172a-454e-91a1-212a5b405cd8"
 					(reference "R6")
 					(unit 1)
 				)
-				(path "/a26094a8-870e-4d79-a298-19a2c7b26655/1ff5d421-dfac-490f-b230-bb532702cb90/95a68da6-4437-469b-a050-26966337937e"
+				(path "/a26094a8-870e-4d79-a298-19a2c7b26655/3b902dd1-f160-4711-ad5c-803c38714d8b/8b541bd0-7703-41c7-b1bc-19a6eec4959f/95a68da6-4437-469b-a050-26966337937e"
 					(reference "R8")
 					(unit 1)
 				)
-				(path "/a26094a8-870e-4d79-a298-19a2c7b26655/1ff5d421-dfac-490f-b230-bb532702cb90/cf5b497f-d460-45bc-b512-00017b3e4ab3"
+				(path "/a26094a8-870e-4d79-a298-19a2c7b26655/3b902dd1-f160-4711-ad5c-803c38714d8b/8b541bd0-7703-41c7-b1bc-19a6eec4959f/cf5b497f-d460-45bc-b512-00017b3e4ab3"
 					(reference "R4")
 					(unit 1)
