File: Half_Bridge.kicad_sch (KiCad schematic)
At the start: 11 parts, among them Q1 SiR622DP, Q2 SiR622DP, Q3 SiR622DP, Q4 SiR622DP, U1 UCC27834DR

Commit message: formatting
Other:
- company: (none) -> Rutgers Capstone ECE 2026-2027
- title: (none) -> Arc Jet PU (Power Unit)
Changed lines of the file:
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@@
 	(generator_version "10.0")
 	(paper "A4")
+	(title_block
+		(title "Arc Jet PU (Power Unit)")
+		(date "2026-10-29")
+		(rev "1.0")
+		(company "Rutgers Capstone ECE 2026-2027")
+		(comment 1 "Mark Tymoshenko mat399@scarletmail.rutgers.edu")
+		(comment 2 "Cy Westbrook")
+	)
 	(text "Bootstrap capacitor should be at least \n20nC/15V * 3 FETs * 10 = 40 nF"
 		(exclude_from_sim no)
@@
 		(instances
 			(project "Arcjet-PPU"
-				(path "/a26094a8-870e-4d79-a298-19a2c7b26655/1ff5d421-dfac-490f-b230-bb532702cb90"
+				(path "/a26094a8-870e-4d79-a298-19a2c7b26655/3b902dd1-f160-4711-ad5c-803c38714d8b/8b541bd0-7703-41c7-b1bc-19a6eec4959f"
 					(reference "C10")
 					(unit 1)
@@
 		(instances
 			(project "Arcjet-PPU"
-				(path "/a26094a8-870e-4d79-a298-19a2c7b26655/1ff5d421-dfac-490f-b230-bb532702cb90"
+				(path "/a26094a8-870e-4d79-a298-19a2c7b26655/3b902dd1-f160-4711-ad5c-803c38714d8b/8b541bd0-7703-41c7-b1bc-19a6eec4959f"
 					(reference "C8")
 					(unit 1)
@@
 		(instances
 			(project "Arcjet-PPU"
-				(path "/a26094a8-870e-4d79-a298-19a2c7b26655/1ff5d421-dfac-490f-b230-bb532702cb90"
+				(path "/a26094a8-870e-4d79-a298-19a2c7b26655/3b902dd1-f160-4711-ad5c-803c38714d8b/8b541bd0-7703-41c7-b1bc-19a6eec4959f"
 					(reference "Q3")
 					(unit 1)
@@
 		(instances
 			(project "Arcjet-PPU"
-				(path "/a26094a8-870e-4d79-a298-19a2c7b26655/1ff5d421-dfac-490f-b230-bb532702cb90"
+				(path "/a26094a8-870e-4d79-a298-19a2c7b26655/3b902dd1-f160-4711-ad5c-803c38714d8b/8b541bd0-7703-41c7-b1bc-19a6eec4959f"
 					(reference "U1")
 					(unit 1)
@@
 		(instances
 			(project "Arcjet-PPU"
-				(path "/a26094a8-870e-4d79-a298-19a2c7b26655/1ff5d421-dfac-490f-b230-bb532702cb90"
+				(path "/a26094a8-870e-4d79-a298-19a2c7b26655/3b902dd1-f160-4711-ad5c-803c38714d8b/8b541bd0-7703-41c7-b1bc-19a6eec4959f"
 					(reference "Q4")
 					(unit 1)
@@
 		(instances
 			(project "Arcjet-PPU"
-				(path "/a26094a8-870e-4d79-a298-19a2c7b26655/1ff5d421-dfac-490f-b230-bb532702cb90"
+				(path "/a26094a8-870e-4d79-a298-19a2c7b26655/3b902dd1-f160-4711-ad5c-803c38714d8b/8b541bd0-7703-41c7-b1bc-19a6eec4959f"
 					(reference "C9")
 					(unit 1)
@@
 		(instances
 			(project "Arcjet-PPU"
-				(path "/a26094a8-870e-4d79-a298-19a2c7b26655/1ff5d421-dfac-490f-b230-bb532702cb90"
+				(path "/a26094a8-870e-4d79-a298-19a2c7b26655/3b902dd1-f160-4711-ad5c-803c38714d8b/8b541bd0-7703-41c7-b1bc-19a6eec4959f"
 					(reference "R1")
 					(unit 1)
@@
 		(instances
 			(project "Arcjet-PPU"
-				(path "/a26094a8-870e-4d79-a298-19a2c7b26655/1ff5d421-dfac-490f-b230-bb532702cb90"
+				(path "/a26094a8-870e-4d79-a298-19a2c7b26655/3b902dd1-f160-4711-ad5c-803c38714d8b/8b541bd0-7703-41c7-b1bc-19a6eec4959f"
 					(reference "#PWR06")
 					(unit 1)
@@
 		(instances
 			(project "Arcjet-PPU"
-				(path "/a26094a8-870e-4d79-a298-19a2c7b26655/1ff5d421-dfac-490f-b230-bb532702cb90"
+				(path "/a26094a8-870e-4d79-a298-19a2c7b26655/3b902dd1-f160-4711-ad5c-803c38714d8b/8b541bd0-7703-41c7-b1bc-19a6eec4959f"
 					(reference "D1")
 					(unit 1)
@@
 		(instances
 			(project "Arcjet-PPU"
-				(path "/a26094a8-870e-4d79-a298-19a2c7b26655/1ff5d421-dfac-490f-b230-bb532702cb90"
+				(path "/a26094a8-870e-4d79-a298-19a2c7b26655/3b902dd1-f160-4711-ad5c-803c38714d8b/8b541bd0-7703-41c7-b1bc-19a6eec4959f"
 					(reference "Q1")
 					(unit 1)
@@
 		(instances
 			(project "Arcjet-PPU"
-				(path "/a26094a8-870e-4d79-a298-19a2c7b26655/1ff5d421-dfac-490f-b230-bb532702cb90"
+				(path "/a26094a8-870e-4d79-a298-19a2c7b26655/3b902dd1-f160-4711-ad5c-803c38714d8b/8b541bd0-7703-41c7-b1bc-19a6eec4959f"
 					(reference "C7")
 					(unit 1)
@@
 		(instances
 			(project "Arcjet-PPU"
-				(path "/a26094a8-870e-4d79-a298-19a2c7b26655/1ff5d421-dfac-490f-b230-bb532702cb90"
+				(path "/a26094a8-870e-4d79-a298-19a2c7b26655/3b902dd1-f160-4711-ad5c-803c38714d8b/8b541bd0-7703-41c7-b1bc-19a6eec4959f"
 					(reference "Q2")
 					(unit 1)
@@
 		(instances
 			(project "Arcjet-PPU"
-				(path "/a26094a8-870e-4d79-a298-19a2c7b26655/1ff5d421-dfac-490f-b230-bb532702cb90"
-					(page "6")
+				(path "/a26094a8-870e-4d79-a298-19a2c7b26655/3b902dd1-f160-4711-ad5c-803c38714d8b/8b541bd0-7703-41c7-b1bc-19a6eec4959f"
+					(page "3")
 				)
 			)
@@
 		(instances
 			(project "Arcjet-PPU"
-				(path "/a26094a8-870e-4d79-a298-19a2c7b26655/1ff5d421-dfac-490f-b230-bb532702cb90"
-					(page "4")
+				(path "/a26094a8-870e-4d79-a298-19a2c7b26655/3b902dd1-f160-4711-ad5c-803c38714d8b/8b541bd0-7703-41c7-b1bc-19a6eec4959f"
+					(page "5")
 				)
 			)
@@
 		(instances
 			(project "Arcjet-PPU"
-				(path "/a26094a8-870e-4d79-a298-19a2c7b26655/1ff5d421-dfac-490f-b230-bb532702cb90"
-					(page "5")
+				(path "/a26094a8-870e-4d79-a298-19a2c7b26655/3b902dd1-f160-4711-ad5c-803c38714d8b/8b541bd0-7703-41c7-b1bc-19a6eec4959f"
+					(page "4")
 				)
 			)
@@
 		(instances
 			(project "Arcjet-PPU"
-				(path "/a26094a8-870e-4d79-a298-19a2c7b26655/1ff5d421-dfac-490f-b230-bb532702cb90"
-					(page "3")
-				)
-			)
+				(path "/a26094a8-870e-4d79-a298-19a2c7b26655/3b902dd1-f160-4711-ad5c-803c38714d8b/8b541bd0-7703-41c7-b1bc-19a6eec4959f"
+					(page "6")
+				)
+			)
